Commit message: load robotiq

File: urdf/ur5_on_table.urdf.xacro (robot description, xacro)
@@ -7,23 +7,21 @@
   <!-- ur5 -->
   <xacro:include filename="$(find ur_description)/urdf/ur5.urdf.xacro" />
-  <!-- arm -->
-  <xacro:ur5_robot prefix="" joint_limited="true"
-    shoulder_pan_lower_limit="${-pi}" shoulder_pan_upper_limit="${pi}"
-    shoulder_lift_lower_limit="${-pi}" shoulder_lift_upper_limit="${pi}"
-    elbow_joint_lower_limit="${-pi}" elbow_joint_upper_limit="${pi}"
-    wrist_1_lower_limit="${-pi}" wrist_1_upper_limit="${pi}"
-    wrist_2_lower_limit="${-pi}" wrist_2_upper_limit="${pi}"
-    wrist_3_lower_limit="${-pi}" wrist_3_upper_limit="${pi}"
-    transmission_hw_interface="$(arg transmission_hw_interface)"
-  />
-  <!-- arm -->
-  <!-- <xacro:ur5_robot prefix="" joint_limited="false" -->
-    <!-- transmission_hw_interface="$(arg transmission_hw_interface)" -->
-  <!-- /> -->
+  <!-- arm joint limited -->
+  <!-- <xacro:ur5_robot prefix="" joint_limited="true" -->
+    <!-- shoulder_pan_lower_limit="${-pi}" shoulder_pan_upper_limit="${pi}" -->
+    <!-- shoulder_lift_lower_limit="${-pi}" shoulder_lift_upper_limit="${pi}" -->
+    <!-- elbow_joint_lower_limit="${-pi}" elbow_joint_upper_limit="${pi}" -->
+    <!-- wrist_1_lower_limit="${-pi}" wrist_1_upper_limit="${pi}" -->
+    <!-- wrist_2_lower_limit="${-pi}" wrist_2_upper_limit="${pi}" -->
+    <!-- wrist_3_lower_limit="${-pi}" wrist_3_upper_limit="${pi}" -->
+    <!-- transmission_hw_interface="$(arg transmission_hw_interface)"/> -->
+  <!-- arm - not joint limited -->
+  <xacro:ur5_robot prefix="" joint_limited="false"
+    transmission_hw_interface="$(arg transmission_hw_interface)"/>
   <!-- Robotiq -->
-  <!-- <xacro:include filename="$(find robotiq_2f_model)/model/robotiq_2f_85.urdf.xacro" /> -->
-  <!-- <xacro:robotiq_2f_85  name="robotiq_2f_85" parent="tool0"> -->
-    <!-- <origin xyz="0.0 0.0 0.0" rpy="0.0 0.0 0.0" /> -->
-  <!-- </xacro:robotiq_2f_85> -->
+  <xacro:include filename="$(find robotiq_2f_model)/model/robotiq_2f_85.urdf.xacro" />
+  <xacro:robotiq_2f_85  name="robotiq_2f_85" parent="tool0">
+    <origin xyz="0.0 0.0 0.0" rpy="0.0 0.0 0.0" />
+  </xacro:robotiq_2f_85>
   <link name="table">
     <visual>

Commit message: replacing robotiq with standin

File: urdf/ur5_on_table.urdf.xacro (robot description, xacro)
@@ -20,8 +20,24 @@
     transmission_hw_interface="$(arg transmission_hw_interface)"/>
   <!-- Robotiq -->
-  <xacro:include filename="$(find robotiq_2f_model)/model/robotiq_2f_85.urdf.xacro" />
-  <xacro:robotiq_2f_85  name="robotiq_2f_85" parent="tool0">
-    <origin xyz="0.0 0.0 0.0" rpy="0.0 0.0 0.0" />
-  </xacro:robotiq_2f_85>
+  <!-- <xacro:include filename="$(find robotiq_2f_model)/model/robotiq_2f_85.urdf.xacro" /> -->
+  <!-- <xacro:robotiq_2f_85  name="robotiq_2f_85" parent="tool0"> -->
+    <!-- <origin xyz="0.0 0.0 0.0" rpy="0.0 0.0 0.0" /> -->
+  <!-- </xacro:robotiq_2f_85> -->
+  <link name="tool_link">
+    <visual>
+      <origin xyz="0 0 0.125"/>
+      <geometry>
+        <cylinder length="0.25" radius="0.06"/>
+      </geometry>
+      <material name="green">
+        <color rgba="0 1 0 1"/>
+      </material>
+    </visual>
+  </link>
+  <joint name="$tool_link_joint" type="fixed">
+    <parent link="tool0"/>
+    <child link="tool_link"/>
+    <origin rpy="0 0 0" xyz="0 0 0"/>
+  </joint>
   <link name="table">
     <visual>

Commit message: Execute demo (#2)
* replacing robotiq with standin

* setting up the demo for execution on UR5

File: urdf/ur5_on_table.urdf.xacro (robot description, xacro)
@@ -8,20 +8,36 @@
   <xacro:include filename="$(find ur_description)/urdf/ur5.urdf.xacro" />
   <!-- arm joint limited -->
-  <!-- <xacro:ur5_robot prefix="" joint_limited="true" -->
-    <!-- shoulder_pan_lower_limit="${-pi}" shoulder_pan_upper_limit="${pi}" -->
-    <!-- shoulder_lift_lower_limit="${-pi}" shoulder_lift_upper_limit="${pi}" -->
-    <!-- elbow_joint_lower_limit="${-pi}" elbow_joint_upper_limit="${pi}" -->
-    <!-- wrist_1_lower_limit="${-pi}" wrist_1_upper_limit="${pi}" -->
-    <!-- wrist_2_lower_limit="${-pi}" wrist_2_upper_limit="${pi}" -->
-    <!-- wrist_3_lower_limit="${-pi}" wrist_3_upper_limit="${pi}" -->
+  <xacro:ur5_robot prefix="" joint_limited="true"
+    shoulder_pan_lower_limit="${-pi}" shoulder_pan_upper_limit="${pi}"
+    shoulder_lift_lower_limit="${-pi}" shoulder_lift_upper_limit="${pi}"
+    elbow_joint_lower_limit="${-pi}" elbow_joint_upper_limit="${pi}"
+    wrist_1_lower_limit="${-pi}" wrist_1_upper_limit="${pi}"
+    wrist_2_lower_limit="${-pi}" wrist_2_upper_limit="${pi}"
+    wrist_3_lower_limit="${-pi}" wrist_3_upper_limit="${pi}"
+    transmission_hw_interface="$(arg transmission_hw_interface)"/>
+  <!-- arm - not joint limited -->
+  <!-- <xacro:ur5_robot prefix="" joint_limited="false" -->
     <!-- transmission_hw_interface="$(arg transmission_hw_interface)"/> -->
-  <!-- arm - not joint limited -->
-  <xacro:ur5_robot prefix="" joint_limited="false"
-    transmission_hw_interface="$(arg transmission_hw_interface)"/>
   <!-- Robotiq -->
-  <xacro:include filename="$(find robotiq_2f_model)/model/robotiq_2f_85.urdf.xacro" />
-  <xacro:robotiq_2f_85  name="robotiq_2f_85" parent="tool0">
-    <origin xyz="0.0 0.0 0.0" rpy="0.0 0.0 0.0" />
-  </xacro:robotiq_2f_85>
+  <!-- <xacro:include filename="$(find robotiq_2f_model)/model/robotiq_2f_85.urdf.xacro" /> -->
+  <!-- <xacro:robotiq_2f_85  name="robotiq_2f_85" parent="tool0"> -->
+    <!-- <origin xyz="0.0 0.0 0.0" rpy="0.0 0.0 0.0" /> -->
+  <!-- </xacro:robotiq_2f_85> -->
+  <link name="tool_link">
+    <visual>
+      <origin xyz="0 0 0.125"/>
+      <geometry>
+        <cylinder length="0.25" radius="0.06"/>
+      </geometry>
+      <material name="green">
+        <color rgba="0 1 0 1"/>
+      </material>
+    </visual>
+  </link>
+  <joint name="$tool_link_joint" type="fixed">
+    <parent link="tool0"/>
+    <child link="tool_link"/>
+    <origin rpy="0 0 0" xyz="0 0 0"/>
+  </joint>
   <link name="table">
     <visual>

Commit message: Use OnlineRobot and fix launch bringup

File: urdf/ur5_on_table.urdf.xacro (robot description, xacro)
@@ -9,19 +9,20 @@
   <!-- arm joint limited -->
   <xacro:ur5_robot prefix="" joint_limited="true"
-    shoulder_pan_lower_limit="${-pi}" shoulder_pan_upper_limit="${pi}"
-    shoulder_lift_lower_limit="${-pi}" shoulder_lift_upper_limit="${pi}"
+    shoulder_pan_lower_limit="${-2*pi}" shoulder_pan_upper_limit="${2*pi}"
+    shoulder_lift_lower_limit="${-2*pi}" shoulder_lift_upper_limit="${2*pi}"
     elbow_joint_lower_limit="${-pi}" elbow_joint_upper_limit="${pi}"
-    wrist_1_lower_limit="${-pi}" wrist_1_upper_limit="${pi}"
-    wrist_2_lower_limit="${-pi}" wrist_2_upper_limit="${pi}"
-    wrist_3_lower_limit="${-pi}" wrist_3_upper_limit="${pi}"
+    wrist_1_lower_limit="${-2*pi}" wrist_1_upper_limit="${2*pi}"
+    wrist_2_lower_limit="${-2*pi}" wrist_2_upper_limit="${2*pi}"
+    wrist_3_lower_limit="${-2*pi}" wrist_3_upper_limit="${2*pi}"
     transmission_hw_interface="$(arg transmission_hw_interface)"/>
   <!-- arm - not joint limited -->
-  <!-- <xacro:ur5_robot prefix="" joint_limited="false" -->
-    <!-- transmission_hw_interface="$(arg transmission_hw_interface)"/> -->
+  <!--<xacro:ur5_robot prefix="" joint_limited="false"
+   transmission_hw_interface="$(arg transmission_hw_interface)"/>-->
   <!-- Robotiq -->
-  <!-- <xacro:include filename="$(find robotiq_2f_model)/model/robotiq_2f_85.urdf.xacro" /> -->
-  <!-- <xacro:robotiq_2f_85  name="robotiq_2f_85" parent="tool0"> -->
-    <!-- <origin xyz="0.0 0.0 0.0" rpy="0.0 0.0 0.0" /> -->
-  <!-- </xacro:robotiq_2f_85> -->
+  <xacro:include filename="$(find robotiq_2f_model)/model/robotiq_2f_85.urdf.xacro" />
+  <xacro:robotiq_2f_85  name="robotiq_2f_85" parent="tool0">
+  <origin xyz="0.0 0.0 0.0" rpy="0.0 0.0 0.0" />
+  </xacro:robotiq_2f_85> -->
+  <!--
   <link name="tool_link">
     <visual>
@@ -40,4 +41,5 @@
     <origin rpy="0 0 0" xyz="0 0 0"/>
   </joint>
+  -->
   <link name="table">
     <visual>

Commit message: pr feedback

File: urdf/ur5_on_table.urdf.xacro (robot description, xacro)
@@ -8,19 +8,19 @@
   <xacro:include filename="$(find ur_description)/urdf/ur5.urdf.xacro" />
   <!-- arm joint limited -->
-  <xacro:ur5_robot prefix="" joint_limited="true"
-    shoulder_pan_lower_limit="${-2*pi}" shoulder_pan_upper_limit="${2*pi}"
-    shoulder_lift_lower_limit="${-2*pi}" shoulder_lift_upper_limit="${2*pi}"
-    elbow_joint_lower_limit="${-pi}" elbow_joint_upper_limit="${pi}"
-    wrist_1_lower_limit="${-2*pi}" wrist_1_upper_limit="${2*pi}"
-    wrist_2_lower_limit="${-2*pi}" wrist_2_upper_limit="${2*pi}"
-    wrist_3_lower_limit="${-2*pi}" wrist_3_upper_limit="${2*pi}"
-    transmission_hw_interface="$(arg transmission_hw_interface)"/>
+  <!-- <xacro:ur5_robot prefix="" joint_limited="true" -->
+    <!-- shoulder_pan_lower_limit="${-pi}" shoulder_pan_upper_limit="${pi}" -->
+    <!-- shoulder_lift_lower_limit="${-pi}" shoulder_lift_upper_limit="${pi}" -->
+    <!-- elbow_joint_lower_limit="${-pi}" elbow_joint_upper_limit="${pi}" -->
+    <!-- wrist_1_lower_limit="${-pi}" wrist_1_upper_limit="${pi}" -->
+    <!-- wrist_2_lower_limit="${-pi}" wrist_2_upper_limit="${pi}" -->
+    <!-- wrist_3_lower_limit="${-pi}" wrist_3_upper_limit="${pi}" -->
+    <!-- transmission_hw_interface="$(arg transmission_hw_interface)"/> -->
   <!-- arm - not joint limited -->
-  <!--<xacro:ur5_robot prefix="" joint_limited="false"
-   transmission_hw_interface="$(arg transmission_hw_interface)"/>-->
+  <xacro:ur5_robot prefix="" joint_limited="false"
+   transmission_hw_interface="$(arg transmission_hw_interface)"/>
   <!-- Robotiq -->
   <xacro:include filename="$(find robotiq_2f_model)/model/robotiq_2f_85.urdf.xacro" />
   <xacro:robotiq_2f_85  name="robotiq_2f_85" parent="tool0">
-  <origin xyz="0.0 0.0 0.0" rpy="0.0 0.0 0.0" />
+    <origin xyz="0.0 0.0 0.0" rpy="0.0 0.0 0.0" />
   </xacro:robotiq_2f_85> -->
   <!--

Commit message: consolodating to one launch file

File: urdf/ur5_on_table.urdf.xacro (robot description, xacro)
@@ -20,9 +20,8 @@
    transmission_hw_interface="$(arg transmission_hw_interface)"/>
   <!-- Robotiq -->
-  <xacro:include filename="$(find robotiq_2f_model)/model/robotiq_2f_85.urdf.xacro" />
-  <xacro:robotiq_2f_85  name="robotiq_2f_85" parent="tool0">
-    <origin xyz="0.0 0.0 0.0" rpy="0.0 0.0 0.0" />
-  </xacro:robotiq_2f_85>
-  <!--
+  <!-- <xacro:include filename="$(find robotiq_2f_model)/model/robotiq_2f_85.urdf.xacro" /> -->
+  <!-- <xacro:robotiq_2f_85  name="robotiq_2f_85" parent="tool0"> -->
+    <!-- <origin xyz="0.0 0.0 0.0" rpy="0.0 0.0 0.0" /> -->
+  <!-- </xacro:robotiq_2f_85> -->
   <link name="tool_link">
     <visual>
@@ -41,5 +40,4 @@
     <origin rpy="0 0 0" xyz="0 0 0"/>
   </joint>
-  -->
   <link name="table">
     <visual>

Commit message: adding robotiq control and improving demo

File: urdf/ur5_on_table.urdf.xacro (robot description, xacro)
@@ -26,7 +26,8 @@
   <link name="tool_link">
     <visual>
-      <origin xyz="0 0 0.125"/>
+      <origin xyz="0 0 0.0875"/>
       <geometry>
-        <cylinder length="0.25" radius="0.06"/>
+        <box size="0.1 0.02 0.175"/>
+        <!-- <cylinder length="0.25" radius="0.06"/> -->
       </geometry>
       <material name="green">
