Commit message: joint specific windup

File: urdf/ur5_on_table_robotiq.urdf.xacro (robot description, xacro)
@@ -20,8 +20,9 @@
    transmission_hw_interface="$(arg transmission_hw_interface)"/>
   <!-- Robotiq -->
-  <!-- <xacro:include filename="$(find robotiq_2f_model)/model/robotiq_2f_85.urdf.xacro" /> -->
-  <!-- <xacro:robotiq_2f_85  name="robotiq_2f_85" parent="tool0"> -->
-    <!-- <origin xyz="0.0 0.0 0.0" rpy="0.0 0.0 0.0" /> -->
-  <!-- </xacro:robotiq_2f_85> -->
+  <xacro:include filename="$(find robotiq_2f_model)/model/robotiq_2f_85.urdf.xacro" />
+  <xacro:robotiq_2f_85  name="robotiq_2f_85" parent="tool0">
+    <origin xyz="0.0 0.0 0.0" rpy="0.0 0.0 0.0" />
+  </xacro:robotiq_2f_85>
+  <!--
   <link name="tool_link">
     <visual>
@@ -40,4 +41,5 @@
     <origin rpy="0 0 0" xyz="0 0 0"/>
   </joint>
+  -->
   <link name="table">
     <visual>

Commit message: Retime traj vel scaling (#5)
* Use OnlineRobot and fix launch bringup
* Implement simple pick/place demo
* adding robotiq control and improving demo
* using velocity and acceleration scaling when retiming the trajectory
* adding moveit_simple to rosinstall

File: urdf/ur5_on_table_robotiq.urdf.xacro (robot description, xacro)
@@ -20,14 +20,14 @@
    transmission_hw_interface="$(arg transmission_hw_interface)"/>
   <!-- Robotiq -->
-  <!-- <xacro:include filename="$(find robotiq_2f_model)/model/robotiq_2f_85.urdf.xacro" /> -->
-  <!-- <xacro:robotiq_2f_85  name="robotiq_2f_85" parent="tool0"> -->
-    <!-- <origin xyz="0.0 0.0 0.0" rpy="0.0 0.0 0.0" /> -->
-  <!-- </xacro:robotiq_2f_85> -->
+  <xacro:include filename="$(find robotiq_2f_model)/model/robotiq_2f_85.urdf.xacro" />
+  <xacro:robotiq_2f_85  name="robotiq_2f_85" parent="tool0">
+    <origin xyz="0.0 0.0 0.0" rpy="0.0 0.0 0.0" />
+  </xacro:robotiq_2f_85>
+  <!--
   <link name="tool_link">
     <visual>
-      <origin xyz="0 0 0.0875"/>
+      <origin xyz="0 0 0.125"/>
       <geometry>
-        <box size="0.1 0.02 0.175"/>
-        <!-- <cylinder length="0.25" radius="0.06"/> -->
+        <cylinder length="0.25" radius="0.06"/>
       </geometry>
       <material name="green">
@@ -41,4 +41,5 @@
     <origin rpy="0 0 0" xyz="0 0 0"/>
   </joint>
+  -->
   <link name="table">
     <visual>
